File: pcb/wasd/wasd.kicad_sch (KiCad schematic)
At the start: 25 parts, among them CN1 S7B-ZR-SM4A-TF(LF)(SN)_C51187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

Commit message: NG | wasd pcb
Parts:
- added H4: MountingHole, MountingHole:MountingHole_3mm, symbol Mechanical:MountingHole
Connections:
- net +5V: now also CN1.6; no longer CN1.2
- net GND: now also CN1.7; no longer CN1.1
- net LED_DATA: now also CN1.1; no longer CN1.7
- net down: now also CN1.4; no longer CN1.5
- net left: now also CN1.5; no longer CN1.4
- net right: now also CN1.2; no longer CN1.6
- net at LED3.2 (DOUT): now also LED4.3 (DIN); no longer LED5.3 (DIN)
- net at LED3.3 (DIN): now also LED2.2 (DOUT); no longer LED4.2 (DOUT)
- net at LED8.3 (DIN): now also LED7.2 (DOUT); no longer LED6.2 (DOUT)
- net at LED5.2 (DOUT): now also LED6.3 (DIN); no longer LED7.3 (DIN)
- new net: LED4.2 (DOUT), LED5.3 (DIN)
- new net: LED6.2 (DOUT), LED7.3 (DIN)
Other:
- moved on the sheet: LED3, LED4, LED6, LED7, LOGO1
