File: pcb/wasd/wasd.kicad_pcb (KiCad board)
At the start: 2 copper layers, 81 x 66.5 mm, 25 parts, among them CN1 S7B-ZR-SM4A-TF(LF)(SN)_C51187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

Commit message: NG | wasd pcb
Parts:
- added H4: MountingHole, MountingHole:MountingHole_3mm, F.Cu at (129.9, 86.0)
- C1, C2, C3, C4, C5, C6, C7, C8, CH2, CH3, CH4, CN1, LOGO1: moved to B.Cu
- moved CH4 107.2 mm to (168.5, 112.6), turned to 180 degrees
- moved C1 99.5 mm to (178.8, 108.2)
- moved LOGO1 87.4 mm to (160.0, 94.0), turned to 180 degrees
- moved C8 83.7 mm to (162.3, 76.8), turned to 180 degrees
- moved H2 81.9 mm to (165.5, 82.9)
- moved CH3 80.6 mm to (142.0, 99.7), turned to 180 degrees
- moved C2 77.9 mm to (157.0, 108.2)
- moved C3 71.9 mm to (153.5, 95.2)
- moved CN1 70.3 mm to (147.9, 120.5), turned to -12 degrees
- moved H3 68.7 mm to (136.3, 126.0)
- moved C7 62.2 mm to (140.0, 76.0), turned to 180 degrees
- moved C4 48.8 mm to (130.5, 95.2)
- moved C5 42.2 mm to (124.0, 95.2)
- moved H1 36.7 mm to (116.9, 82.7)
- moved LED7 35.0 mm to (143.4, 71.4)
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Connections:
- CN1 pad 1: GND -> LED_DATA
- CN1 pad 2: +5V -> right
- CN1 pad 4: left -> down
- CN1 pad 5: down -> left
- CN1 pad 6: right -> +5V
- CN1 pad 7: LED_DATA -> GND
- LED3 pad 3: Net-(LED3-DIN) -> Net-(LED2-DOUT)
- LED4 pad 2: Net-(LED3-DIN) -> Net-(LED4-DOUT)
- LED4 pad 3: Net-(LED2-DOUT) -> Net-(LED3-DOUT)
- LED5 pad 3: Net-(LED3-DOUT) -> Net-(LED4-DOUT)
- LED6 pad 3: Net-(LED6-DIN) -> Net-(LED5-DOUT)
- LED7 pad 2: Net-(LED6-DIN) -> Net-(LED7-DOUT)
- LED7 pad 3: Net-(LED5-DOUT) -> Net-(LED6-DOUT)
- LED8 pad 3: Net-(LED6-DOUT) -> Net-(LED7-DOUT)
Routing:
- net +5V: track 0.00 -> 246.9 mm, vias 0 -> 9
- net up: track 0.00 -> 57.2 mm, vias 0 -> 2
- net Net-(LED6-DOUT): track 0.00 -> 56.5 mm, vias 0 -> 2
- net left: track 0.00 -> 52.1 mm
- net LED_DATA: track 0.00 -> 39.7 mm, vias 0 -> 2
- net down: track 0.00 -> 23.9 mm
- net Net-(LED2-DOUT): track 0.00 -> 17.7 mm
- net Net-(LED5-DOUT): track 0.00 -> 16.0 mm
- net Net-(LED3-DOUT): track 0.00 -> 15.9 mm
- net Net-(LED1-DOUT): track 0.00 -> 15.8 mm
- net Net-(LED7-DOUT): track 0.00 -> 15.7 mm
- net right: track 0.00 -> 11.4 mm
- net Net-(LED4-DOUT): track 0.00 -> 7.67 mm
- net GND: track 0.00 -> 1.64 mm, vias 0 -> 30
- added copper zone on B.Cu, net GND
- added copper zone on F.Cu, net GND
Other:
- board size 81 x 66.5 mm -> 81 x 69.2 mm
- board text added: "v1"
