File: pcb/usb-ext/usb-ext.kicad_pcb (KiCad board)
At the start: 2 copper layers, 21.4 x 31.3 mm, 4 parts

Commit message: NG | Splitfox PCB Placement
Connections:
- USB1 pad 4: Net-(USB1-GND) -> GND
- USB1 pad 5: unconnected-(USB1-EH-Pad5) -> GND
- USB2 pad 4: Net-(USB1-GND) -> GND
- USB2 pad 5: unconnected-(USB2-Pad5) -> GND
- USB2 pad 6: unconnected-(USB2-Pad6) -> GND
- USB2 pad 7: unconnected-(USB2-Pad7) -> GND
- USB2 pad 8: unconnected-(USB2-Pad8) -> GND
Routing:
- net Net-(USB1-GND): vias 7 -> 0
- net GND: vias 0 -> 7
- added copper zone on B.Cu, net GND
- added copper zone on F.Cu, net GND
- removed copper zone on B.Cu, net Net-(USB1-GND)
- removed copper zone on F.Cu, net Net-(USB1-GND)
Changed lines of the file:
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@@
 	(net 2 "Net-(USB1-D+)")
 	(net 3 "Net-(USB1-VBUS)")
-	(net 4 "Net-(USB1-GND)")
-	(net 5 "unconnected-(USB2-Pad7)")
-	(net 6 "unconnected-(USB2-Pad8)")
-	(net 7 "unconnected-(USB1-EH-Pad5)")
-	(net 8 "unconnected-(USB2-Pad5)")
-	(net 9 "unconnected-(USB2-Pad6)")
+	(net 4 "GND")
 	(footprint "MountingHole:MountingHole_3mm"
 		(layer "F.Cu")
@@
 			(size 1 2.5)
 			(layers "F.Cu" "F.Paste" "F.Mask")
-			(net 4 "Net-(USB1-GND)")
+			(net 4 "GND")
 			(pinfunction "GND")
 			(pintype "input")
@@
 			(layers "*.Cu" "*.Mask")
 			(remove_unused_layers no)
-			(net 7 "unconnected-(USB1-EH-Pad5)")
+			(net 4 "GND")
 			(pinfunction "EH")
 			(pintype "input")
@@
 			(layers "*.Cu" "*.Mask")
 			(remove_unused_layers no)
-			(net 7 "unconnected-(USB1-EH-Pad5)")
+			(net 4 "GND")
 			(pinfunction "EH")
 			(pintype "input")
@@
 			(size 1.2 2.5)
 			(layers "F.Cu" "F.Paste" "F.Mask")
-			(net 4 "Net-(USB1-GND)")
+			(net 4 "GND")
 			(pinfunction "GND")
 			(pintype "unspecified")
@@
 			(layers "*.Cu" "*.Mask")
 			(remove_unused_layers no)
-			(net 8 "unconnected-(USB2-Pad5)")
+			(net 4 "GND")
 			(pinfunction "5")
 			(pintype "unspecified")
@@
 			(layers "*.Cu" "*.Mask")
 			(remove_unused_layers no)
-			(net 9 "unconnected-(USB2-Pad6)")
+			(net 4 "GND")
 			(pinfunction "6")
 			(pintype "unspecified")
@@
 			(layers "*.Cu" "*.Mask")
 			(remove_unused_layers no)
-			(net 5 "unconnected-(USB2-Pad7)")
+			(net 4 "GND")
 			(pinfunction "7")
 			(pintype "unspecified")
@@
 			(layers "*.Cu" "*.Mask")
 			(remove_unused_layers no)
-			(net 6 "unconnected-(USB2-Pad8)")
+			(net 4 "GND")
 			(pinfunction "8")
 			(pintype "unspecified")
@@
 		(sheetname "Root")
 		(sheetfile "usb-ext.kicad_sch")
-		(attr through_hole)
+		(attr through_hole exclude_from_bom)
 		(fp_poly
 			(pts
@@
 	(zone
 		(net 4)
-		(net_name "Net-(USB1-GND)")
+		(net_name "GND")
 		(layers "F&B.Cu")
 		(name "GND")
