File: pcb/usb-ext/usb-ext.kicad_pcb (KiCad board)
At the start: 2 copper layers, 21.4 x 31.3 mm, 4 parts

Commit message: NG | It's done-ish, pcb tweaks, assembly
Parts:
- moved USB1 0.98 mm to (154.9, 87.1)
Routing:
- net Net-(USB1-D+): track 12.6 -> 11.3 mm
- net Net-(USB1-VBUS): track 11.7 -> 10.6 mm
- net Net-(USB1-D-): track 12.4 -> 11.4 mm
Other:
- board size 21.4 x 31.3 mm -> 21.4 x 30.3 mm
Changed lines of the file:
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@@
 	(title_block
 		(title "usb-ext")
-		(date "2025-02-11")
+		(date "2025-02-12")
 		(rev "v1")
 		(company "Speedy Labs")
@@
 	(footprint "easyeda:USB-SMD_AM180CB"
 		(layer "F.Cu")
-		(at 154.9 86.1475 180)
+		(at 154.9 87.125 180)
 		(property "Reference" "USB1"
 			(at -0.1 -3.8525 180)
@@
 	)
 	(gr_arc
-		(start 164.764285 81.700001)
-		(mid 164.941062 81.773224)
-		(end 165.014285 81.950001)
+		(start 164.764285 82.677501)
+		(mid 164.941063 82.750722)
+		(end 165.014285 82.927501)
 		(stroke
 			(width 0.25)
@@
 	)
 	(gr_line
-		(start 145.064285 81.700001)
-		(end 164.764285 81.700001)
-		(stroke
-			(width 0.25)
-			(type default)
-		)
-		(layer "Edge.Cuts")
-	)
-	(gr_line
-		(start 165.014285 81.950001)
+		(start 145.064285 82.677501)
+		(end 164.764285 82.677501)
+		(stroke
+			(width 0.25)
+			(type default)
+		)
+		(layer "Edge.Cuts")
+	)
+	(gr_line
+		(start 165.014285 82.927501)
 		(end 165.014285 110.000001)
 		(stroke
@@
 	)
 	(gr_line
-		(start 144.814285 81.950001)
+		(start 144.814285 82.927501)
 		(end 144.814285 110)
 		(stroke
@@
 	)
 	(gr_arc
-		(start 144.814285 81.950001)
-		(mid 144.887508 81.773224)
-		(end 145.064285 81.700001)
+		(start 144.814285 82.927501)
+		(mid 144.88751 82.750726)
+		(end 145.064285 82.677501)
 		(stroke
 			(width 0.25)
@@
 	)
 	(segment
-		(start 152 90.1775)
-		(end 152 95.7925)
-		(width 1)
+		(start 152.09 94.61)
+		(end 152.09 91.5)
+		(width 0.8)
 		(layer "F.Cu")
 		(net 1)
 	)
 	(segment
-		(start 152 95.7925)
-		(end 153.91 97.7025)
-		(width 1)
+		(start 153.9 89.69)
+		(end 152.09 91.5)
+		(width 0.8)
 		(layer "F.Cu")
 		(net 1)
 	)
 	(segment
-		(start 153.91 97.7025)
-		(end 153.91 98.3525)
-		(width 1)
+		(start 153.9 88.505)
+		(end 153.9 89.69)
+		(width 0.8)
 		(layer "F.Cu")
 		(net 1)
 	)
 	(segment
-		(start 153.9 87.5275)
-		(end 153.9 88.2775)
-		(width 1)
+		(start 153.91 96.43)
+		(end 152.09 94.61)
+		(width 0.8)
 		(layer "F.Cu")
 		(net 1)
 	)
 	(segment
-		(start 153.9 88.2775)
-		(end 152 90.1775)
-		(width 1)
+		(start 153.91 98.3525)
+		(end 153.91 96.43)
+		(width 0.8)
 		(layer "F.Cu")
 		(net 1)
 	)
 	(segment
-		(start 158 95.5125)
-		(end 155.91 97.6025)
-		(width 1)
+		(start 155.9 89.82)
+		(end 157.69 91.61)
+		(width 0.8)
 		(layer "F.Cu")
 		(net 2)
 	)
 	(segment
-		(start 155.9 88.2775)
-		(end 158 90.3775)
-		(width 1)
+		(start 155.9 88.505)
+		(end 155.9 89.82)
+		(width 0.8)
 		(layer "F.Cu")
 		(net 2)
 	)
 	(segment
-		(start 158 90.3775)
-		(end 158 95.5125)
-		(width 1)
+		(start 155.91 98.3525)
+		(end 155.91 96.42)
+		(width 0.8)
 		(layer "F.Cu")
 		(net 2)
 	)
 	(segment
-		(start 155.91 97.6025)
-		(end 155.91 98.3525)
-		(width 1)
+		(start 157.69 94.64)
+		(end 157.69 91.61)
+		(width 0.8)
 		(layer "F.Cu")
 		(net 2)
 	)
 	(segment
-		(start 155.9 87.5275)
-		(end 155.9 88.2775)
-		(width 1)
+		(start 155.91 96.42)
+		(end 157.69 94.64)
+		(width 0.8)
 		(layer "F.Cu")
 		(net 2)
 	)
 	(segment
-		(start 150.3 88.6275)
-		(end 150.3 97.2425)
+		(start 150.49 89.415)
+		(end 150.49 97.4325)
 		(width 2)
 		(layer "F.Cu")
@@
 	)
 	(segment
-		(start 151.4 87.5275)
-		(end 150.3 88.6275)
+		(start 150.49 97.4325)
+		(end 151.41 98.3525)
 		(width 2)
 		(layer "F.Cu")
@@
 	)
 	(segment
-		(start 150.3 97.2425)
-		(end 151.41 98.3525)
+		(start 151.4 88.505)
+		(end 150.49 89.415)
 		(width 2)
 		(layer "F.Cu")
@@
 	)
 	(via
-		(at 155 85)
+		(at 154.85 86.01)
 		(size 0.6)
 		(drill 0.3)
