File: pcb/usb-ext/usb-ext.kicad_sch (KiCad schematic)
At the start: 4 parts

Commit message: NG | Splitfox PCB Placement
Connections:
- net GND: now reaches USB1.4 (GND), USB2.4 (GND)
- net GND: now also USB1.5 (EH), USB2.5, USB2.6, USB2.7, USB2.8
